File: board/revision-1/army-simple-fc.kicad_pcb (KiCad board)
At the start: 2 copper layers, 70 x 25 mm, 73 parts, among them J1 Conn_01x03, J10 Conn_01x03, J11 Conn_01x03, J12 Conn_01x03, J13 Conn_01x03, J14 Conn_01x03, J15 Conn_01x03, J16 Conn_01x03, J17 Conn_01x03, J18 Conn_01x06, J2 Conn_01x03, J3 Conn_01x03, J4 Conn_01x03, J5 Conn_01x06, J7 Conn_01x03, J8 Conn_01x03, J9 Conn_01x03, Q1 BC817-40, Q2 BC817-40, Q3 BC817-40, Q4 BC817-40, Q5 BC817-40, U1 MCP1703Ax-120xxTT, U3 STM32G070KBTx, X1 TagConnect_TC2030

Commit message: Майже всунув.
Parts:
- moved J10 46.9 mm to (163.2, 91.6)
- moved J2 38.0 mm to (209.8, 86.0)
- moved J9 36.7 mm to (165.2, 97.2)
- moved Q1 35.3 mm to (170.5, 112.8)
- moved R12 35.3 mm to (174.8, 113.0)
- moved R14 35.3 mm to (173.2, 113.0)
- moved J5 31.5 mm to (195.8, 86.0)
- moved Q5 28.4 mm to (180.1, 90.0)
- moved R31 28.3 mm to (182.8, 90.0)
- moved R27 28.2 mm to (184.0, 89.8)
- moved Q2 27.4 mm to (180.9, 104.8)
- moved R15 27.4 mm to (183.8, 104.8)
- moved R13 27.4 mm to (185.4, 104.8)
- moved J3 24.3 mm to (202.8, 86.0)
- moved R17 23.6 mm to (180.8, 110.6), turned to 180 degrees
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Connections:
- R4 pad 2: /UART1.TX -> /UART3.TX
- R5 pad 2: /UART1.RX -> /UART3.RX
- R7 pad 2: /UART3.TX -> /UART1.TX
- R8 pad 2: /UART3.RX -> /UART1.RX
Routing:
- net Net-(J14-Pin_3): track 0.00 -> 26.1 mm
- net Net-(D4-A): track 16.5 -> 41.5 mm
- net Net-(D5-A): track 11.1 -> 31.0 mm
- net Net-(J13-Pin_3): track 0.00 -> 17.9 mm
- net Net-(J12-Pin_3): track 4.41 -> 16.6 mm
- net Net-(J2-Pin_2): track 0.00 -> 11.6 mm, vias 0 -> 1
- net /NRST: track 0.00 -> 10.6 mm, vias 0 -> 1
- net Net-(D6-A): track 6.93 -> 17.5 mm
- net /ADC1_IN5: track 0.00 -> 10.3 mm
- net /I2C2.SCL: track 0.00 -> 8.07 mm
- net Net-(J5-Pin_3): track 0.00 -> 7.97 mm
- net Net-(J3-Pin_2): track 0.00 -> 6.97 mm
- net /ADC1_IN10: track 0.00 -> 5.88 mm
- net Net-(J15-Pin_2): track 0.00 -> 5.47 mm
- net /SWDIO: track 0.00 -> 5.09 mm, vias 0 -> 1
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Other:
- board text added: "G"
- board text added: "PWM2"
- board text added: "PWM3"
- board text added: "PWM4"
- board text added: "S"
- board text added: "V"

Commit message: Майже закінчив.
Parts:
- removed the J3 at (202.8, 86.0)
- added C7: 0.1uF, Capacitor_SMD:C_0603_1608Metric, F.Cu at (191.8, 103.9)
- C1: value 100uF,10V -> 100uF; footprint Capacitor_Tantalum_SMD:CP_EIA-6032-20_AVX-F -> Capacitor_SMD:C_1206_3216Metric
- J2: footprint Connector_JST:JST_PH_B2B-PH-K_1x02_P2.00mm_Vertical -> Connector_JST:JST_PH_B3B-PH-K_1x03_P2.00mm_Vertical
- moved J11 48.5 mm to (211.4, 86.0)
- moved Q5 22.8 mm to (176.9, 97.0), turned to 90 degrees
- moved FID1 21.8 mm to (155.6, 105.4)
- moved FID2 21.8 mm to (222.4, 83.6)
- moved R32 21.3 mm to (179.4, 97.5), turned to 90 degrees
- moved R23 20.9 mm to (200.2, 89.0), turned to 0 degrees
- moved R31 18.8 mm to (176.7, 99.7), turned to 180 degrees
- moved J7 16.8 mm to (163.8, 91.5)
- moved R30 16.6 mm to (176.7, 101.2), turned to 180 degrees
- moved R17 14.3 mm to (185.8, 103.9), turned to 180 degrees
- moved R20 12.5 mm to (171.3, 104.0), turned to 180 degrees
- moved Q1 11.9 mm to (168.0, 101.2), turned to 90 degrees
- moved R29 10.7 mm to (180.8, 103.1)
- moved R19 10.4 mm to (167.8, 104.0), turned to 180 degrees
- moved Q2 10.1 mm to (171.5, 101.1), turned to 90 degrees
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- renumbered C4 to C2, C5 to C3, C3 to C4, C2 to C5, J9 to J10, J10 to J11, J15 to J12, J16 to J13, J8 to J14, J17 to J15, J18 to J16, J11 to J3, J12 to J4, J13 to J5, J14 to J6, J4 to J7, J5 to J8, J7 to J9, Q4 to Q3, Q5 to Q4, Q3 to Q5, R3 to R1, R24 to R10, R4 to R11, R5 to R12, R7 to R13, R8 to R14, R2 to R15, R6 to R16, R12 to R17, R13 to R18, R14 to R19, R1 to R2, R15 to R20, R17 to R21, R18 to R22, R19 to R23, R26 to R24, R27 to R25, R30 to R26, R31 to R27, R16 to R28, R32 to R29, R10 to R3, R25 to R30, R29 to R31, R28 to R32, R9 to R4, R11 to R5, R20 to R6, R21 to R7, R22 to R8, R23 to R9, U3 to U2
Connections:
- D3 pad 1: /TIM3_CH1 -> /TIM14_CH1
- D3 pad 3: /TIM3_CH2 -> /TIM3_CH4
- D3 pad 5: /TIM3_CH4 -> /TIM3_CH2
- D3 pad 6: /TIM14_CH1 -> /TIM3_CH1
- J16 pad 4: /SPI1_MOSI -> /SPI1_CLK
- J16 pad 6: /SPI1_CLK -> /SPI1_MOSI
- J9 pad 1: Net-(J7-Pin_1) -> GND
- J9 pad 2: GND -> Net-(J9-Pin_2)
- J9 pad 3: Net-(J7-Pin_3) (its old number) -> Net-(J9-Pin_3)
- Q1 pad 3: Net-(J7-Pin_1) -> Net-(J9-Pin_3)
- Q2 pad 3: Net-(J7-Pin_3) (its old number) -> Net-(J9-Pin_2)
- R17 pad 1: /WINCH-DOWN -> /WINCH-UP
- R18 pad 1: /WINCH-UP -> /WINCH-DOWN
- R2 pad 1: Net-(J3-Pin_2) -> Net-(J2-Pin_3)
- R28 pad 1: /UART2.RX -> /UART2.TX
- R29 pad 1: /UART2.TX -> /UART2.RX
- X1 pad 6: /UART2.TX -> unconnected-(X1-SWO/PRG_RX-Pad6)
Routing:
- net +5V: track 21.3 -> 120.4 mm
- net /SPI1_MOSI: track 0.00 -> 38.7 mm, vias 0 -> 1
- net /SPI1_MISO: track 0.00 -> 36.9 mm, vias 0 -> 1
- net /SPI1_CLK: track 0.00 -> 35.7 mm, vias 0 -> 1
- net /SPI1_CS: track 0.00 -> 32.7 mm, vias 0 -> 1
- net +3.3V: track 0.00 -> 32.7 mm, vias 0 -> 2
- net Net-(J7-Pin_3): track 0.00 -> 26.7 mm, vias 0 -> 1
- net Net-(J7-Pin_4): track 0.00 -> 26.6 mm, vias 0 -> 1
- net Net-(J14-Pin_4): track 0.00 -> 23.9 mm, vias 0 -> 1
- net Net-(J14-Pin_3): track 0.00 -> 22.9 mm, vias 0 -> 1
- net Net-(Q1-B): track 0.00 -> 22.7 mm
- net Net-(J10-Pin_4): track 0.00 -> 21.4 mm, vias 0 -> 1
- net /UART4.RX: track 0.00 -> 20.0 mm, vias 0 -> 2
- net /UART4.TX: track 0.00 -> 19.6 mm, vias 0 -> 2
- net Net-(J10-Pin_3): track 0.00 -> 19.1 mm, vias 0 -> 1
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
Commit message: Завершив. Почнемо збирати гербери.
Parts:
- moved R1 0.45 mm to (199.3, 98.5)
- moved R3 0.36 mm to (197.7, 98.5)
- moved R30 0.30 mm to (176.7, 101.5)
- moved R23 0.30 mm to (199.9, 89.0)
- moved R7 0.30 mm to (199.9, 90.6)
- moved R9 0.30 mm to (199.9, 92.2)
- moved C4 0.28 mm to (196.1, 98.5)
- moved R31 0.20 mm to (176.7, 99.9)
- moved R32 0.14 mm to (179.5, 97.6)
- moved C5 0.10 mm to (192.3, 89.7)
- moved R11 0.10 mm to (180.8, 99.9)
- moved R24 0.10 mm to (176.7, 94.4)
- moved R26 0.10 mm to (176.7, 92.9)
- moved C2 0.10 mm to (196.9, 101.4)
- moved Q5 0.10 mm to (176.9, 97.1)
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Routing:
- net GND: track 4.09 -> 6.55 mm, vias 17 -> 21
- net /TIM14_CH1: track 14.1 -> 16.2 mm, vias 2 -> 0
- net /UART4.TX: track 19.6 -> 17.9 mm
- net +5V: track 120.4 -> 118.9 mm
- net /UART4.RX: track 20.0 -> 18.7 mm
- net Net-(J14-Pin_3): track 22.9 -> 21.7 mm
- net Net-(J6-Pin_3): track 25.9 -> 27.1 mm
- net Net-(J5-Pin_3): track 17.3 -> 18.1 mm
- net Net-(J2-Pin_2): track 15.4 -> 14.7 mm
- net /TIM3_CH4: track 8.76 -> 9.44 mm
- net Net-(J7-Pin_3): track 26.7 -> 26.2 mm
Other:
- board text added: "5V"
- board text added: "ADC"
- board text added: "ARMY-SIMPLE-FC v1.0"
- board text added: "BEEPER"
- board text added: "DEBUG"
- board text added: "GPS"
- board text added: "MOTOR1"
- board text added: "MOTOR2"
- board text added: "MOTOR3"
- board text added: "MOTOR4"
- board text added: "RECEIVER"
- board text added: "SPI"
- board text added: "STARTER"
- board text added: "THROTT"
- board text added: "VTX SA"
- board text added: "VTX SW"
- board text added: "WINCH"
- board text removed: "G"
- board text removed: "PWM1"
- board text removed: "PWM2"
- board text removed: "PWM3"
- board text removed: "PWM4"
- board text removed: "S"
- board text removed: "V"
