File: board/revision-1/army-simple-fc.kicad_sch (KiCad schematic)
At the start: 73 parts, among them J1 Conn_01x03, J10 Conn_01x03, J11 Conn_01x03, J12 Conn_01x03, J13 Conn_01x03, J14 Conn_01x03, J15 Conn_01x03, J16 Conn_01x03, J17 Conn_01x03, J18 Conn_01x06, J2 Conn_01x03, J3 Conn_01x03, J4 Conn_01x03, J5 Conn_01x06, J7 Conn_01x03, J8 Conn_01x03, J9 Conn_01x03, Q1 BC817-40, Q2 BC817-40, Q3 BC817-40, Q4 BC817-40, Q5 BC817-40, U1 MCP1703Ax-120xxTT, U3 STM32G070KBTx, X1 TagConnect_TC2030

Commit message: Майже всунув.
Connections:
- net UART1.RX: now also R8.2; no longer R5.2
- net UART1.TX: now also R7.2; no longer R4.2
- net UART3.RX: now also R5.2; no longer R8.2
- net UART3.TX: now also R4.2; no longer R7.2
Changed lines of the file:
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@@
 	)
 	(label "UART1.RX"
-		(at 64.77 102.87 180)
+		(at 63.5 140.97 180)
 		(fields_autoplaced yes)
 		(effects
@@
 	)
 	(label "UART3.TX"
-		(at 63.5 138.43 180)
+		(at 64.77 100.33 180)
 		(fields_autoplaced yes)
 		(effects
@@
 	)
 	(label "UART3.RX"
-		(at 63.5 140.97 180)
+		(at 64.77 102.87 180)
 		(fields_autoplaced yes)
 		(effects
@@
 	)
 	(label "UART1.TX"
-		(at 64.77 100.33 180)
-		(fields_autoplaced yes)
-		(effects
+		(at 63.5 138.43 180)
+		(fields_autoplaced yes)
+		(effects

Commit message: Майже закінчив.
Parts:
- removed C1: 100uF,10V, Capacitor_Tantalum_SMD:CP_EIA-6032-20_AVX-F, symbol Device:C_Polarized
- removed J2, J3: Conn_01x03, Connector_JST:JST_PH_B2B-PH-K_1x02_P2.00mm_Vertical, symbol Connector_Generic:Conn_01x02
- added C1: 100uF, Capacitor_SMD:C_1206_3216Metric, symbol Device:C
- added C7: 0.1uF, Capacitor_SMD:C_0603_1608Metric, symbol Device:C
- added J2: Conn_01x03, Connector_JST:JST_PH_B3B-PH-K_1x03_P2.00mm_Vertical, symbol Connector_Generic:Conn_01x03
- renumbered C4 to C2, C5 to C3, C3 to C4, C2 to C5, J9 to J10, J10 to J11, J15 to J12, J16 to J13, J8 to J14, J17 to J15, J18 to J16, J11 to J3, J12 to J4, J13 to J5, J14 to J6, J4 to J7, J5 to J8, J7 to J9, Q4 to Q3, Q5 to Q4, Q3 to Q5, R3 to R1, R24 to R10, R4 to R11, R5 to R12, R7 to R13, R8 to R14, R2 to R15, R6 to R16, R12 to R17, R13 to R18, R14 to R19, R1 to R2, R15 to R20, R17 to R21, R18 to R22, R19 to R23, R26 to R24, R27 to R25, R30 to R26, R31 to R27, R16 to R28, R32 to R29, R10 to R3, R25 to R30, R29 to R31, R28 to R32, R9 to R4, R11 to R5, R20 to R6, R21 to R7, R22 to R8, R23 to R9, U3 to U2
Connections:
- net +5V: now also C1.1
- net GND: now also J9.1 (Pin_1), C1.2, C7.2, J2.1 (Pin_1); no longer J9.2 (Pin_2)
- net NRST: now also C7.1
- net SPI1_CLK: now also J16.4 (Pin_4); no longer J16.6 (Pin_6)
- net SPI1_MOSI: now also J16.6 (Pin_6); no longer J16.4 (Pin_4)
- net TIM14_CH1: now also D3.1 (IO1); no longer D3.6 (IO5)
- net TIM3_CH1: now also D3.6 (IO5); no longer D3.1 (IO1)
- net TIM3_CH2: now also D3.5 (IO4); no longer D3.3 (IO2)
- net TIM3_CH4: now also D3.3 (IO2); no longer D3.5 (IO4)
- net UART2.RX: now also R29.1; no longer R28.1
- net UART2.TX: now also R28.1; no longer R29.1, X1.6 (SWO/PRG_RX)
- net WINCH-DOWN: now also R18.1; no longer R17.1
- net WINCH-UP: now also R17.1; no longer R18.1
- net at R1.1: now also J2.2 (Pin_2)
- net at Q2.3 (C): now also J9.2 (Pin_2); no longer J9.3 (Pin_3)
- net at Q1.3 (C): now also J9.3 (Pin_3); no longer J9.1 (Pin_1)
- net at R2.1: now also J2.3 (Pin_3)
Other:
- note added: "ADC1"
- note added: "ADC2"
- note removed: "(PUTTY/DEBUG)"
- note removed: "25V"
- note removed: "42V"
- note removed: "Optional?"
- note removed: "TCK"
- note removed: "TMS"
- moved on the sheet: C4, D3, D5, D6, D7, J11, J16, J4, J5, J6, J9, R1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

Commit message: Завершив. Почнемо збирати гербери.
Other:
- company: (none) -> DROPLA
- title: (none) -> ARMY-SIMPLE-FC
Changed lines of the file:
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@@
 	(generator_version "8.0")
 	(paper "A4")
+	(title_block
+		(title "ARMY-SIMPLE-FC")
+		(date "2024-10-11")
+		(rev "1.0")
+		(company "DROPLA")
+	)
 	(junction
 		(at 53.34 69.85)
